File: Leonardo_Rev3e.kicad_sch (KiCad schematic)
At the start: 56 parts, among them IC1 REG1117-5, IC2 LMV358IDGKR, J1 USBMICRO, J2 8x1F-H8.5, J3 8x1F-H8.5, J4 6x1F-H8.5, T1 FDN340P, U1 ATMEGA32U4-XUMU, U2 ATMEGA32U4-XUAU, U3 LP2985-33DBVR, Y1 16MHz KX-7

Commit message: chore: adapt for forked repo
Other:
- company: (none) -> Further adapted by Aanas Sayed
- title: (none) -> Leonardo Board
Changed lines of the file:
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@@
 	(paper "A3")
 	(title_block
-		(date "2023-02-27")
+		(title "Leonardo Board")
+		(date "2024-12-17")
 		(rev "3e")
+		(company "Further adapted by Aanas Sayed")
+		(comment 1 "Ported to KiCad by Ronan LE MEILLAT (https://github.com/eltorio/leonardo)")
+		(comment 2 "Arduino © Leonardo (https://content.arduino.cc/assets/Leonardo-reference.zip)")
+		(comment 3 "Adapted from")
 	)
 	(junction

Commit message: chore: clean up footprints
Parts:
- C1, C13, C2, C22, C6, C9: value 100n -> 100n-16V; footprint Leonardo_Rev3e:C0603-ROUND -> Capacitor_SMD:C_0603_1608Metric_Pad1.08x0.95mm_HandSolder; Digikey_ref 399-C0603C104J4RAC7867CT-ND -> (none); Manufacturer Kemet -> KEMET; Manufacturer_ref C0603C104J4RAC7867 -> (none); Mfg Part No (none) -> C0603C104J4RAC7867; Vendor (none) -> DIGIKEY; Vendor Part No (none) -> 399-C0603C104J4RAC7867CT-ND
- C10, C12, C8: Digikey_ref 399-3708-1-ND -> (none); Manufacturer Kemet -> KEMET; Manufacturer_ref T491B106M016AT -> (none); Mfg Part No (none) -> T491B106M016AT; Vendor (none) -> DIGIKEY; Vendor Part No (none) -> 399-3708-1-ND
- C11, C14, C5, C7: footprint Leonardo_Rev3e:C0603-ROUND -> Capacitor_SMD:C_0603_1608Metric_Pad1.08x0.95mm_HandSolder; Digikey_ref 399-C0603C105K4RAC7411CT-ND -> (none); Manufacturer Kemet -> KEMET; Manufacturer_ref C0603C105K4RAC7411 -> (none); Mfg Part No (none) -> C0603C105K4RAC7411; Vendor (none) -> DIGIKEY; Vendor Part No (none) -> 399-C0603C105K4RAC7411CT-ND
- C3, C4: footprint Leonardo_Rev3e:C0603-ROUND -> Capacitor_SMD:C_0603_1608Metric_Pad1.08x0.95mm_HandSolder; Digikey_ref 399-14962-1-ND -> (none); Manufacturer Kemet -> KEMET; Manufacturer_ref C0603C220K5RAC7867 -> (none); Mfg Part No (none) -> C0603C220K5RAC7867; Vendor (none) -> DIGIKEY; Vendor Part No (none) -> 399-14962-1-ND
- D+0, D-0, FID1, FID2, FID3, GND0, VUSB0: now left out of the parts list
- D1: footprint Leonardo_Rev3e:SMB -> Diode_SMD:D_SMB; symbol Leonardo_Rev3e:DIODE-SMB -> Device:D
- D2: footprint Leonardo_Rev3e:MINIMELF -> Diode_SMD:D_SOD-123; symbol Leonardo_Rev3e:DIODE-MINIMELF -> Device:D; Digikey_ref 1N4148WTPMSCT-ND -> (none); Manufacturer_ref 1N4148W-TP -> (none); Mfg Part No (none) -> 1N4148W-TP; Vendor (none) -> DIGIKEY; Vendor Part No (none) -> 1N4148WTPMSCT-ND
- F1: Digikey_ref MF-MSMF050-2CT-ND -> (none); Manufacturer Bourns -> BOURNS; Manufacturer_ref MF-MSMF050-2 -> (none); Mfg Part No (none) -> MF-MSMF050-2; Vendor (none) -> DIGIKEY; Vendor Part No (none) -> MF-MSMF050-2CT-ND
- IC1: footprint Leonardo_Rev3e:SOT223 -> Package_TO_SOT_SMD:SOT-223; Digikey_ref REG1117-5-ND -> (none); Manufacturer TI -> TEXAS INSTRUMENTS; Manufacturer_ref REG1117-5 -> (none); Mfg Part No (none) -> REG1117-5; Vendor (none) -> DIGIKEY; Vendor Part No (none) -> REG1117-5-ND
- IC2: footprint Leonardo_Rev3e:MSOP08 -> Package_SO:MSOP-8_3x3mm_P0.65mm; Digikey_ref LMV358IDGKR -> (none); Manufacturer TI -> TEXAS INSTRUMENTS; Manufacturer_ref 296-13455-1-ND -> (none); Mfg Part No (none) -> 296-13455-1-ND; Vendor (none) -> DIGIKEY; Vendor Part No (none) -> LMV358IDGKR
- ICSP0: Digikey_ref A128860-ND -> (none); Manufacturer_ref 5-146486-3 -> (none); Mfg Part No (none) -> 5-146486-3; Vendor (none) -> DIGIKEY; Vendor Part No (none) -> A128860-ND
- J1: Digikey_ref 609-4618-1-ND -> (none); Manufacturer Amphenol -> AMPHENOL; Manufacturer_ref 10118194-0001LF -> (none); Mfg Part No (none) -> 10118194-0001LF; Vendor (none) -> DIGIKEY; Vendor Part No (none) -> 609-4618-1-ND
- J2, J3: Digikey_ref S7041-ND -> (none); Manufacturer Sullins -> SULLINS; Manufacturer_ref PPPC081LFBN-RC -> (none); Mfg Part No (none) -> PPPC081LFBN-RC; Vendor (none) -> DIGIKEY; Vendor Part No (none) -> S7041-ND
- J4: Digikey_ref S7039-ND -> (none); Manufacturer Sullins -> SULLINS; Manufacturer_ref PPPC061LFBN-RC -> (none); Mfg Part No (none) -> PPPC061LFBN-RC; Vendor (none) -> DIGIKEY; Vendor Part No (none) -> S7039-ND
- JP1: Digikey_ref S7043-ND -> (none); Manufacturer Sullins -> SULLINS; Manufacturer_ref PPPC101LFBN-RC -> (none); Mfg Part No (none) -> PPPC101LFBN-RC; Vendor (none) -> DIGIKEY; Vendor Part No (none) -> S7043-ND
- JP2: Digikey_ref SAM15134-ND -> (none); Manufacturer Samtex -> SAMTEC; Manufacturer_ref DW-02-07-T-S-200 -> (none); Mfg Part No (none) -> DW-02-07-T-S-200; Vendor (none) -> DIGIKEY; Vendor Part No (none) -> SAM15134-ND
- L0: Digikey_ref 160-1428-1-ND -> (none); Manufacturer Lite-on -> LITE-ON; Manufacturer_ref LTST-C171KSKT -> (none); Mfg Part No (none) -> LTST-C171KSKT; Vendor (none) -> DIGIKEY; Vendor Part No (none) -> 160-1428-1-ND
- L1, L2: footprint Leonardo_Rev3e:0805 -> Resistor_SMD:R_0805_2012Metric_Pad1.20x1.40mm_HandSolder; Digikey_ref MH2029-300YCT-ND -> (none); Manufacturer Bourns -> BOURNS; Manufacturer_ref MH2029-300Y -> (none); Mfg Part No (none) -> MH2029-300Y; Vendor (none) -> DIGIKEY; Vendor Part No (none) -> MH2029-300YCT-ND
- ON0: Digikey_ref 160-1426-1-ND -> (none); Manufacturer Lite-on -> LITE-ON; Manufacturer_ref LTST-C171KGKT -> (none); Mfg Part No (none) -> LTST-C171KGKT; Vendor (none) -> DIGIKEY; Vendor Part No (none) -> 160-1426-1-ND
- R1: footprint Leonardo_Rev3e:R0603-ROUND -> Resistor_SMD:R_0603_1608Metric_Pad0.98x0.95mm_HandSolder; Digikey_ref CR0603-FX-1004ELFCT-ND -> (none); Manufacturer Bourns -> BOURNS; Manufacturer_ref CR0603-FX-1004ELF -> (none); Mfg Part No (none) -> CR0603-FX-1004ELF; Vendor (none) -> DIGIKEY; Vendor Part No (none) -> CR0603-FX-1004ELFCT-ND
- R2, R3: footprint Leonardo_Rev3e:R0402 -> Resistor_SMD:R_0402_1005Metric_Pad0.72x0.64mm_HandSolder; now not fitted
- R4: footprint Leonardo_Rev3e:R0603-ROUND -> Resistor_SMD:R_0603_1608Metric_Pad0.98x0.95mm_HandSolder; Digikey_ref CR0603-FX-1002ELFCT-ND -> (none); Manufacturer Bourns -> BOURNS; Manufacturer_ref CR0603-FX-1002ELF -> (none); Mfg Part No (none) -> CR0603-FX-1002ELF; Vendor (none) -> DIGIKEY; Vendor Part No (none) -> CR0603-FX-1002ELFCT-ND
- RESET0: Digikey_ref 2223-TS07-667-30-BK-160-SMT-TRCT-ND -> (none); Manufacturer_ref TS07-667-30-BK-160-SMT-TR -> (none); Mfg Part No (none) -> TS07-667-30-BK-160-SMT-TR; Vendor (none) -> DIGIKEY; Vendor Part No (none) -> 2223-TS07-667-30-BK-160-SMT-TRCT-ND
- RN1: Digikey_ref CAY16-1002F4LFCT-ND -> (none); Manufacturer Bourns -> BOURNS; Manufacturer_ref CAY16-1002F4LF -> (none); Mfg Part No (none) -> CAY16-1002F4LF; Vendor (none) -> DIGIKEY; Vendor Part No (none) -> CAY16-1002F4LFCT-ND
- RN2: Digikey_ref CAY16-1001F4LFCT-ND -> (none); Manufacturer Bourns -> BOURNS; Manufacturer_ref CAY16-1001F4LF -> (none); Mfg Part No (none) -> CAY16-1001F4LF; Vendor (none) -> DIGIKEY; Vendor Part No (none) -> CAY16-1001F4LFCT-ND
- RN3: Digikey_ref CAY16-22R0F4LFCT-ND -> (none); Manufacturer Bourns -> BOURNS; Manufacturer_ref CAY16-22R0F4LF -> (none); Mfg Part No (none) -> CAY16-22R0F4LF; Vendor (none) -> DIGIKEY; Vendor Part No (none) -> CAY16-22R0F4LFCT-ND
- RX0, TX0: Digikey_ref 160-1426-1-ND -> (none); Manufacturer Lite-on -> LITE-ON; Manufacturer_ref LTST-C171KSKT -> (none); Mfg Part No (none) -> LTST-C171KSKT; Vendor (none) -> DIGIKEY; Vendor Part No (none) -> 160-1428-1-ND
- T1: footprint Leonardo_Rev3e:SOT-23 -> Package_TO_SOT_SMD:SOT-23; Digikey_ref 4518-FDN340PCT-ND -> (none); Manufacturer_ref FDN340P -> (none); Mfg Part No (none) -> FDN340P; Vendor (none) -> DIGIKEY; Vendor Part No (none) -> 4518-FDN340PCT-ND
- U1: Digikey_ref ATMEGA32U4-MU-ND -> (none); Manufacturer Microchip -> MICROCHIP TECHNOLOGY; Manufacturer_ref ATMEGA32U4-MU -> (none); Mfg Part No (none) -> ATMEGA32U4-MU; Vendor (none) -> DIGIKEY; Vendor Part No (none) -> ATMEGA32U4-MU-ND
- U2: Digikey_ref ATMEGA32U4-AU-ND -> (none); Manufacturer Microchip -> MICROCHIP TECHNOLOGY; Manufacturer_ref ATMEGA32U4-AU -> (none); Mfg Part No (none) -> ATMEGA32U4-AU; Vendor (none) -> DIGIKEY; Vendor Part No (none) -> ATMEGA32U4-AU-ND
- U3: footprint Leonardo_Rev3e:SOT23-DBV -> Package_TO_SOT_SMD:SOT-23-5; Digikey_ref LP2985IM5-3.3CT-ND -> (none); Manufacturer TI -> TEXAS INSTRUMENTS; Manufacturer_ref LP2985IM5-3.3 -> (none); Mfg Part No (none) -> LP2985IM5-3.3; Vendor (none) -> DIGIKEY; Vendor Part No (none) -> LP2985IM5-3.3CT-ND
- Z1, Z2: footprint Leonardo_Rev3e:CT_CN0603 -> Resistor_SMD:R_0603_1608Metric_Pad0.98x0.95mm_HandSolder; Digikey_ref CG0603MLC-05ECT-ND -> (none); Manufacturer Bourns -> BOURNS; Manufacturer_ref CG0603MLC-05E -> (none); Mfg Part No (none) -> CG0603MLC-05E; Vendor (none) -> DIGIKEY; Vendor Part No (none) -> CG0603MLC-05ECT-ND
Connections:
- net +5V: now also D2.1 (K); no longer D2.C
- net 3x2M_NM: now also D1.2 (A); no longer D1.A, U2.P$1 (PAD)
- net GATE_CMD: now also T1.1 (G); no longer T1.3 (G)
- net RESET: now also D2.2 (A); no longer D2.A
- net VIN: now also D1.1 (K); no longer D1.C
- net VUSB: now also T1.3 (D); no longer T1.1 (D)

Commit message: feat: use def. sym/foot and customised BOM and silkscreen
Parts:
- C1, C13, C2, C22, C6, C9: Manufacturer KEMET -> WURTH ELEKTRONIK; Mfg Part No C0603C104J4RAC7867 -> 885012206046; Vendor DIGIKEY -> MOUSER; Vendor Part No 399-C0603C104J4RAC7867CT-ND -> 710-885012206046
- C10, C12, C8: value 10u -> 10u-16V; footprint Leonardo_Rev3e:SMC_B -> Capacitor_SMD:C_1206_3216Metric_Pad1.33x1.80mm_HandSolder; symbol Leonardo_Rev3e:CPOL-EUSMCB -> Device:C; Manufacturer KEMET -> WURTH ELEKTRONIK; Mfg Part No T491B106M016AT -> 885012208041; Vendor DIGIKEY -> MOUSER; Vendor Part No 399-3708-1-ND -> 710-885012208041
- C11, C14, C5, C7: value 1uF -> 1uF-16V; Manufacturer KEMET -> WURTH ELEKTRONIK; Mfg Part No C0603C105K4RAC7411 -> 885012206052; Vendor DIGIKEY -> MOUSER; Vendor Part No 399-C0603C105K4RAC7411CT-ND -> 710-885012206052
- C3, C4: value 22p -> 22p-10V; Manufacturer KEMET -> WURTH ELEKTRONIK; Mfg Part No C0603C220K5RAC7867 -> 885012006004; Vendor DIGIKEY -> MOUSER; Vendor Part No 399-14962-1-ND -> 710-885012006004
- D+0, D-0, FID1, FID2, FID3, GND0, VUSB0: now not fitted
- D1: value M7 -> PMEG6020AELR; footprint Diode_SMD:D_SMB -> Diode_SMD:Nexperia_CFP3_SOD-123W; Manufacturer (none) -> NEXPERIA; Mfg Part No (none) -> PMEG6020AELRX; Vendor (none) -> MOUSER; Vendor Part No (none) -> 771-PMEG6020AELRX
- D2: value 1N4148W-TP -> PMEG4005EH; footprint Diode_SMD:D_SOD-123 -> Diode_SMD:D_SOD-123F; Manufacturer MCC -> NEXPERIA; Mfg Part No 1N4148W-TP -> PMEG4005EH,115; Vendor DIGIKEY -> MOUSER; Vendor Part No 1N4148WTPMSCT-ND -> 771-PMEG4005EH-T/R
- EXTPOWER0: footprint Leonardo_Rev3e:POWERSUPPLY_DC-21MM -> Leonardo_Rev3e:BarrelJack_Horizontal_Wurth_694108301002; Manufacturer (none) -> WURTH ELEKTRONIK; Mfg Part No (none) -> 694108301002; Vendor (none) -> MOUSER; Vendor Part No (none) -> 710-694108301002
- F1: value MF-MSMF050-2 500mA -> 500mA; footprint Leonardo_Rev3e:L1812 -> Fuse:Fuse_1812_4532Metric_Pad1.30x3.40mm_HandSolder; Manufacturer BOURNS -> BEL FUSE; Mfg Part No MF-MSMF050-2 -> 0ZCG0050FF2C; Vendor DIGIKEY -> MOUSER; Vendor Part No MF-MSMF050-2CT-ND -> 530-0ZCG0050FF2C
- IC1: value REG1117-5 -> LDI1117-05H; Manufacturer TEXAS INSTRUMENTS -> DIOTEC SEMICONDUCTOR; Mfg Part No REG1117-5 -> LDI1117-05H; Vendor DIGIKEY -> MOUSER; Vendor Part No REG1117-5-ND -> 637-LDI1117-05H
- IC2: value LMV358IDGKR -> LM358LVIDGKR; Mfg Part No 296-13455-1-ND -> LM358LVIDGKR; Vendor DIGIKEY -> MOUSER; Vendor Part No LMV358IDGKR -> 595-LM358LVIDGKR
- ICSP0: Manufacturer TE -> WURTH ELEKTRONIK; Mfg Part No 5-146486-3 -> 61300621121; Vendor DIGIKEY -> MOUSER; Vendor Part No A128860-ND -> 710-61300621121
- J1: footprint Leonardo_Rev3e:10118194-0001LF -> Leonardo_Rev3e:Micro_USB_2.0_SMT_Type_B_Wurth_629105150521; symbol Leonardo_Rev3e:USBMICRO -> Connector:USB_B_Micro; Manufacturer AMPHENOL -> WURTH ELEKTRONIK; Mfg Part No 10118194-0001LF -> 629105150521; Vendor DIGIKEY -> MOUSER; Vendor Part No 609-4618-1-ND -> 710-629105150521
- J2, J3: Manufacturer SULLINS -> WURTH ELEKTRONIK; Mfg Part No PPPC081LFBN-RC -> 61300811821; Vendor DIGIKEY -> MOUSER; Vendor Part No S7041-ND -> 710-61300811821
- J4: Manufacturer SULLINS -> WURTH ELEKTRONIK; Mfg Part No PPPC061LFBN-RC -> 61300611821; Vendor DIGIKEY -> MOUSER; Vendor Part No S7039-ND -> 710-61300611821
- JP1: Manufacturer SULLINS -> WURTH ELEKTRONIK; Mfg Part No PPPC101LFBN-RC -> 61301011821; Vendor DIGIKEY -> MOUSER; Vendor Part No S7043-ND -> 710-61301011821
- JP2: Manufacturer SAMTEC -> WURTH ELEKTRONIK; Mfg Part No DW-02-07-T-S-200 -> 61300211121; Vendor DIGIKEY -> MOUSER; Vendor Part No SAM15134-ND -> 710-61300211121; now not fitted
- L0, RX0, TX0: Manufacturer LITE-ON -> WURTH ELEKTRONIK; Mfg Part No LTST-C171KSKT -> 150080YS75000; Vendor DIGIKEY -> MOUSER; Vendor Part No 160-1428-1-ND -> 710-150080YS75000
- L1, L2: Manufacturer BOURNS -> WURTH ELEKTRONIK; Mfg Part No MH2029-300Y -> 74279206; Vendor DIGIKEY -> MOUSER; Vendor Part No MH2029-300YCT-ND -> 710-74279206
- ON0: Manufacturer LITE-ON -> WURTH ELEKTRONIK; Mfg Part No LTST-C171KGKT -> 150080GS75000; Vendor DIGIKEY -> MOUSER; Vendor Part No 160-1426-1-ND -> 710-150080GS75000
- R1: Vendor DIGIKEY -> MOUSER; Vendor Part No CR0603-FX-1004ELFCT-ND -> 652-CR0603FX-1004ELF
- R2, R3: value NM -> 0; Manufacturer (none) -> YAGEO; Mfg Part No (none) -> RC0603FR-070RL; Vendor (none) -> MOUSER; Vendor Part No (none) -> 603-RC0603FR-070RL
- R4: Manufacturer BOURNS -> KAMAYA; Mfg Part No CR0603-FX-1002ELF -> RMC1/16-103JTP; Vendor DIGIKEY -> MOUSER; Vendor Part No CR0603-FX-1002ELFCT-ND -> 791-RMC1/16103JTP
- RESET0: value TS07-667-30-BK-160-SMT-TR -> 431181015816; footprint Leonardo_Rev3e:TS07 -> Leonardo_Rev3e:PushButton_Wurth_431181015816; symbol Leonardo_Rev3e:TS07 -> Switch:SW_Push_Shielded; Manufacturer CUI -> WURTH ELEKTRONIK; Mfg Part No TS07-667-30-BK-160-SMT-TR -> 431181015816; Vendor DIGIKEY -> MOUSER; Vendor Part No 2223-TS07-667-30-BK-160-SMT-TRCT-ND -> 710-431181015816
- RN1: value 10K -> 10k; footprint Leonardo_Rev3e:CAY16 -> Resistor_SMD:R_Cat16-4; Vendor DIGIKEY -> MOUSER; Vendor Part No CAY16-1002F4LFCT-ND -> 652-CAY16-1002F4LF
- RN2: value 1K -> 1k; footprint Leonardo_Rev3e:CAY16 -> Resistor_SMD:R_Cat16-4; Vendor DIGIKEY -> MOUSER; Vendor Part No CAY16-1001F4LFCT-ND -> 652-CAY16-1001F4LF
- RN3: footprint Leonardo_Rev3e:CAY16 -> Resistor_SMD:R_Cat16-4; Vendor DIGIKEY -> MOUSER; Vendor Part No CAY16-22R0F4LFCT-ND -> 652-CAY16-22R0F4LF
- T1: value FDN340P -> NXV65UP; Manufacturer UMW -> NEXPERIA; Mfg Part No FDN340P -> NXV65UPR; Vendor DIGIKEY -> MOUSER; Vendor Part No 4518-FDN340PCT-ND -> 771-NXV65UPR
- U1: value ATMEGA32U4-XUMU -> ATMEGA32U4-MU; Vendor DIGIKEY -> MOUSER; Vendor Part No ATMEGA32U4-MU-ND -> 556-ATMEGA32U4-MU
- U2: value ATMEGA32U4-XUAU -> ATMEGA32U4-AU; Vendor DIGIKEY -> MOUSER; Vendor Part No ATMEGA32U4-AU-ND -> 556-ATMEGA32U4-AU; now not fitted
- U3: value LP2985-33DBVR -> LDI559-3.3EN; Manufacturer TEXAS INSTRUMENTS -> DIOTEC SEMICONDUCTOR; Mfg Part No LP2985IM5-3.3 -> LDI559-3.3EN; Vendor DIGIKEY -> MOUSER; Vendor Part No LP2985IM5-3.3CT-ND -> 637-LDI559-3.3EN
- Y1: value 16MHz KX-7 -> 16MHz; Manufacturer (none) -> GEYER ELECTRONIC AMERICA, INC.; Mfg Part No (none) -> 12.88722; Vendor (none) -> DIGIKEY; Vendor Part No (none) -> 4983-12.88722CT-ND
- Z1, Z2: Manufacturer BOURNS -> WURTH ELEKTRONIK; Mfg Part No CG0603MLC-05E -> 82306050029; Vendor DIGIKEY -> MOUSER; Vendor Part No CG0603MLC-05ECT-ND -> 710-82306050029
Connections:
- net +5V: now also C12.1; no longer C12.+
- net 3x2M_NM: now also C10.2, C12.2, C8.2, EXTPOWER0.2, RESET0.SH (B); no longer C10.-, C12.-, C8.-, D1.2 (A), EXTPOWER0.1, RESET0.4
- net D+: now also J1.3 (D+); no longer J1.P3 (D+)
- net D-: now also J1.2 (D-); no longer J1.P2 (D-)
- net RESET: no longer RESET0.3
- net UGND: now also J1.5 (GND); no longer J1.P5 (GND)
- net USBID: now also J1.4 (ID); no longer J1.P4 (ID)
- net VIN: now also C10.1; no longer C10.+, EXTPOWER0.2
- net VUSB: now also C8.1; no longer C8.+
- net XUSB: now also J1.1 (VBUS); no longer J1.P1 (VBUS)
- removed net 5-GND: RESET0.5 (5-GND)
- new net: D1.2 (A), EXTPOWER0.1
- no-connect marks 0 -> 1
Other:
- moved on the sheet: D1, EXTPOWER0, RN3A, RN3D
