File: Leonardo_Rev3e.kicad_sch (KiCad schematic)
At the start: 56 parts, among them IC1 LDI1117-05H, IC2 LM358LVIDGKR, J1 USBMICRO, J2 8x1F-H8.5, J3 8x1F-H8.5, J4 6x1F-H8.5, T1 NXV65UP, U1 ATMEGA32U4-MU, U2 ATMEGA32U4-AU, U3 LDI559-3.3EN, Y1 16MHz

Commit message: chore: update bom
Parts:
- D+0, D-0, FID1, FID2, FID3, GND0, VUSB0: now fitted
- EXTPOWER0: value POWERSUPPLY_DC21MMX -> POWERSUPPLY_DC21MM
- L1, L2: value MH2029-300Y -> 74279206
- RN1: value 10k -> 10K
- RN2: value 1k -> 1K
- Z1, Z2: value CG0603MLC-05E -> 82306050029
Changed lines of the file:
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@@
 		(in_bom no)
 		(on_board yes)
-		(dnp yes)
+		(dnp no)
 		(property "Reference" "VUSB0"
 			(at 90.17 187.452 0)
@@
 			)
 		)
-		(property "Value" "MH2029-300Y"
+		(property "Value" "74279206"
 			(at 96.52 125.73 0)
 			(effects
@@
 		(in_bom no)
 		(on_board yes)
-		(dnp yes)
+		(dnp no)
 		(property "Reference" "FID2"
 			(at 46.99 17.78 0)
@@
 		(in_bom no)
 		(on_board yes)
-		(dnp yes)
+		(dnp no)
 		(property "Reference" "D+0"
 			(at 83.312 223.52 0)
@@
 			)
 		)
-		(property "Value" "CG0603MLC-05E"
+		(property "Value" "82306050029"
 			(at 92.71 246.38 0)
 			(effects
@@
 		(in_bom no)
 		(on_board yes)
-		(dnp yes)
+		(dnp no)
 		(property "Reference" "GND0"
 			(at 82.55 253.492 0)
@@
 			)
 		)
-		(property "Value" "MH2029-300Y"
+		(property "Value" "74279206"
 			(at 58.42 222.25 0)
 			(effects
@@
 			)
 		)
-		(property "Value" "10k"
+		(property "Value" "10K"
 			(at 174.498 233.68 0)
 			(effects
@@
 			)
 		)
-		(property "Value" "10k"
+		(property "Value" "10K"
 			(at 347.98 155.702 0)
 			(effects
@@
 			)
 		)
-		(property "Value" "1k"
+		(property "Value" "1K"
 			(at 369.57 86.36 0)
 			(effects
@@
 		(in_bom no)
 		(on_board yes)
-		(dnp yes)
+		(dnp no)
 		(property "Reference" "D-0"
 			(at 103.378 218.44 0)
@@
 			)
 		)
-		(property "Value" "10k"
+		(property "Value" "10K"
 			(at 88.138 93.98 0)
 			(effects
@@
 			)
 		)
-		(property "Value" "1k"
+		(property "Value" "1K"
 			(at 328.422 86.36 0)
 			(effects
@@
 			)
 		)
-		(property "Value" "POWERSUPPLY_DC21MMX"
+		(property "Value" "POWERSUPPLY_DC21MM"
 			(at 59.69 27.94 0)
 			(effects
@@
 		(in_bom no)
 		(on_board yes)
-		(dnp yes)
+		(dnp no)
 		(property "Reference" "FID3"
 			(at 54.61 17.78 0)
@@
 			)
 		)
-		(property "Value" "1k"
+		(property "Value" "1K"
 			(at 351.282 88.9 0)
 			(effects
@@
 			)
 		)
-		(property "Value" "10k"
+		(property "Value" "10K"
 			(at 168.402 223.52 0)
 			(effects
@@
 		(in_bom no)
 		(on_board yes)
-		(dnp yes)
+		(dnp no)
 		(property "Reference" "FID1"
 			(at 39.37 17.78 0)
@@
 			)
 		)
-		(property "Value" "CG0603MLC-05E"
+		(property "Value" "82306050029"
 			(at 102.87 246.38 0)
 			(effects
@@
 			)
 		)
-		(property "Value" "1k"
+		(property "Value" "1K"
 			(at 338.582 88.9 0)
 			(effects

Commit message: chore: remove trailing whitespaces in BOM
Parts:
- C1, C10, C11, C12, C13, C14, C2, C22, C3, C4, C5, C6, C7, C8, C9, EXTPOWER0, ICSP0, J1, J2, J3, J4, JP1, JP2, L0, L1, L2, ON0, RESET0, RX0, TX0, Z1, Z2: Manufacturer WURTH ELEKTRONIK -> WURTH ELEKTRONIK
Changed lines of the file:
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@@
 			)
 		)
-		(property "Manufacturer" "WURTH ELEKTRONIK "
+		(property "Manufacturer" "WURTH ELEKTRONIK"
 			(at 181.61 236.22 0)
 			(effects
@@
 			)
 		)
-		(property "Manufacturer" "WURTH ELEKTRONIK "
+		(property "Manufacturer" "WURTH ELEKTRONIK"
 			(at 318.77 236.22 0)
 			(effects
@@
 			)
 		)
-		(property "Manufacturer" "WURTH ELEKTRONIK "
+		(property "Manufacturer" "WURTH ELEKTRONIK"
 			(at 54.61 109.22 0)
 			(effects
@@
 			)
 		)
-		(property "Manufacturer" "WURTH ELEKTRONIK "
+		(property "Manufacturer" "WURTH ELEKTRONIK"
 			(at 100.33 124.46 0)
 			(effects
@@
 			)
 		)
-		(property "Manufacturer" "WURTH ELEKTRONIK "
+		(property "Manufacturer" "WURTH ELEKTRONIK"
 			(at 57.15 119.38 0)
 			(effects
@@
 			)
 		)
-		(property "Manufacturer" "WURTH ELEKTRONIK "
+		(property "Manufacturer" "WURTH ELEKTRONIK"
 			(at 194.31 86.36 0)
 			(effects
@@
 			)
 		)
-		(property "Manufacturer" "WURTH ELEKTRONIK "
+		(property "Manufacturer" "WURTH ELEKTRONIK"
 			(at 69.85 132.08 0)
 			(effects
@@
 			)
 		)
-		(property "Manufacturer" "WURTH ELEKTRONIK "
+		(property "Manufacturer" "WURTH ELEKTRONIK"
 			(at 341.63 93.98 0)
 			(effects
@@
 			)
 		)
-		(property "Manufacturer" "WURTH ELEKTRONIK "
+		(property "Manufacturer" "WURTH ELEKTRONIK"
 			(at 161.29 30.48 0)
 			(effects
@@
 			)
 		)
-		(property "Manufacturer" "WURTH ELEKTRONIK "
+		(property "Manufacturer" "WURTH ELEKTRONIK"
 			(at 153.67 231.14 0)
 			(effects
@@
 			)
 		)
-		(property "Manufacturer" "WURTH ELEKTRONIK "
+		(property "Manufacturer" "WURTH ELEKTRONIK"
 			(at 123.19 234.95 0)
 			(effects
@@
 			)
 		)
-		(property "Manufacturer" "WURTH ELEKTRONIK "
+		(property "Manufacturer" "WURTH ELEKTRONIK"
 			(at 110.49 88.9 0)
 			(effects
@@
 			)
 		)
-		(property "Manufacturer" "WURTH ELEKTRONIK "
+		(property "Manufacturer" "WURTH ELEKTRONIK"
 			(at 85.09 137.16 0)
 			(effects
@@
 			)
 		)
-		(property "Manufacturer" "WURTH ELEKTRONIK "
+		(property "Manufacturer" "WURTH ELEKTRONIK"
 			(at 87.63 238.76 0)
 			(effects
@@
 			)
 		)
-		(property "Manufacturer" "WURTH ELEKTRONIK "
+		(property "Manufacturer" "WURTH ELEKTRONIK"
 			(at 54.61 223.52 0)
 			(effects
@@
 			)
 		)
-		(property "Manufacturer" "WURTH ELEKTRONIK "
+		(property "Manufacturer" "WURTH ELEKTRONIK"
 			(at 273.05 246.38 0)
 			(effects
@@
 			)
 		)
-		(property "Manufacturer" "WURTH ELEKTRONIK "
+		(property "Manufacturer" "WURTH ELEKTRONIK"
 			(at 133.35 236.22 0)
 			(effects
@@
 			)
 		)
-		(property "Manufacturer" "WURTH ELEKTRONIK "
+		(property "Manufacturer" "WURTH ELEKTRONIK"
 			(at 97.79 144.78 0)
 			(effects
@@
 			)
 		)
-		(property "Manufacturer" "WURTH ELEKTRONIK "
+		(property "Manufacturer" "WURTH ELEKTRONIK"
 			(at 85.09 46.99 0)
 			(effects
@@
 			)
 		)
-		(property "Manufacturer" "WURTH ELEKTRONIK "
+		(property "Manufacturer" "WURTH ELEKTRONIK"
 			(at 354.33 93.98 0)
 			(effects
@@
 			)
 		)
-		(property "Manufacturer" "WURTH ELEKTRONIK "
+		(property "Manufacturer" "WURTH ELEKTRONIK"
 			(at 46.99 68.58 0)
 			(effects
@@
 			)
 		)
-		(property "Manufacturer" "WURTH ELEKTRONIK "
+		(property "Manufacturer" "WURTH ELEKTRONIK"
 			(at 49.53 33.02 0)
 			(effects
@@
 			)
 		)
-		(property "Manufacturer" "WURTH ELEKTRONIK "
+		(property "Manufacturer" "WURTH ELEKTRONIK"
 			(at 100.33 88.9 0)
 			(effects
@@
 			)
 		)
-		(property "Manufacturer" "WURTH ELEKTRONIK "
+		(property "Manufacturer" "WURTH ELEKTRONIK"
 			(at 191.77 30.48 0)
 			(effects
@@
 			)
 		)
-		(property "Manufacturer" "WURTH ELEKTRONIK "
+		(property "Manufacturer" "WURTH ELEKTRONIK"
 			(at 74.93 215.9 0)
 			(effects
@@
 			)
 		)
-		(property "Manufacturer" "WURTH ELEKTRONIK "
+		(property "Manufacturer" "WURTH ELEKTRONIK"
 			(at 92.71 73.66 0)
 			(effects
@@
 			)
 		)
-		(property "Manufacturer" "WURTH ELEKTRONIK "
+		(property "Manufacturer" "WURTH ELEKTRONIK"
 			(at 57.15 205.74 0)
 			(effects
@@
 			)
 		)
-		(property "Manufacturer" "WURTH ELEKTRONIK "
+		(property "Manufacturer" "WURTH ELEKTRONIK"
 			(at 331.47 93.98 0)
 			(effects
@@
 			)
 		)
-		(property "Manufacturer" "WURTH ELEKTRONIK "
+		(property "Manufacturer" "WURTH ELEKTRONIK"
 			(at 163.83 86.36 0)
 			(effects
@@
 			)
 		)
-		(property "Manufacturer" "WURTH ELEKTRONIK "
+		(property "Manufacturer" "WURTH ELEKTRONIK"
 			(at 97.79 238.76 0)
 			(effects
@@
 			)
 		)
-		(property "Manufacturer" "WURTH ELEKTRONIK "
+		(property "Manufacturer" "WURTH ELEKTRONIK"
 			(at 130.81 44.45 0)
 			(effects
@@
 			)
 		)
-		(property "Manufacturer" "WURTH ELEKTRONIK "
+		(property "Manufacturer" "WURTH ELEKTRONIK"
 			(at 367.03 99.06 0)
 			(effects
